File: Documentation/Electrical/Schematics/Sources/ElectricalSchematicforStorage - Ducks/ElectricalSchematicforStorage.kicad_sch (KiCad schematic)
At the start: 2 parts

Commit message: addressed changes
Other:
- note added: "Micro Maestro 6-Channel USB Servo Controller"
- note removed: "Micro Masetro 6-Channel USB Servo Controller"
Changed lines of the file:
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@@
     (effects (font (size 1.27 1.27)) (justify left bottom))
   )
-  (text "Micro Masetro 6-Channel\nUSB Servo Controller\n" (at 60.96 71.12 0)
+  (text "Micro Maestro 6-Channel\nUSB Servo Controller\n" (at 60.96 71.12 0)
     (effects (font (size 1.27 1.27)) (justify left bottom))
   )
