File: Documentation/Electrical/Schematics/Sources/SortingSubsystem/SortingSubsystem/SortingSubsystem.kicad_sch (KiCad schematic)
At the start: 4 parts, among them M1 Motor_Servo, U1 TB9051FTG

Commit message: updated electrical schematic
Parts:
- gave numbers to parts that had none: 1
Changed lines of the file:
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@@
   )
   (polyline (pts (xy 312.674 165.354) (xy 312.674 143.51))
-    (stroke (width 0) (type default) (color 0 0 0 0))
+    (stroke (width 0) (type solid) (color 0 0 0 0))
   )
   (wire (pts (xy 95.25 76.2) (xy 120.65 76.2))
@@
     (stroke (width 0) (type default) (color 0 0 0 0))
   )
-  (polyline (pts (xy 279.654 165.1) (xy 312.674 165.354))
-    (stroke (width 0) (type default) (color 0 0 0 0))
-  )
   (polyline (pts (xy 107.95 153.67) (xy 107.95 186.69))
     (stroke (width 0) (type default) (color 0 0 0 0))
@@
     (stroke (width 0) (type default) (color 0 0 0 0))
   )
-  (polyline (pts (xy 279.4 143.51) (xy 279.654 165.1))
-    (stroke (width 0) (type default) (color 0 0 0 0))
+  (polyline (pts (xy 279.4 143.51) (xy 279.4 165.1))
+    (stroke (width 0) (type solid) (color 0 0 0 0))
   )
   (wire (pts (xy 313.69 158.75) (xy 341.63 158.75))
@@
   )
   (polyline (pts (xy 279.4 143.51) (xy 312.674 143.51))
-    (stroke (width 0) (type default) (color 0 0 0 0))
+    (stroke (width 0) (type solid) (color 0 0 0 0))
   )
   (wire (pts (xy 113.03 152.4) (xy 113.03 154.94))
@@
     (stroke (width 0) (type default) (color 0 0 0 0))
   )
+  (polyline (pts (xy 279.4 165.1) (xy 312.42 165.1))
+    (stroke (width 0) (type solid) (color 0 0 0 0))
+  )
   (wire (pts (xy 205.74 152.4) (xy 217.17 152.4))
     (stroke (width 0) (type default) (color 0 0 0 0))
@@
   )
   (label "pin 46" (at 113.03 184.15 0)
+    (effects (font (size 1.27 1.27)) (justify left bottom))
+  )
+  (label "DC Motor with encoder" (at 285.75 143.51 0)
     (effects (font (size 1.27 1.27)) (justify left bottom))
   )
@@
   (symbol (lib_id "Motor:Motor_DC") (at 297.18 152.4 0) (unit 1)
     (in_bom yes) (on_board yes) (fields_autoplaced)
-    (property "Reference" "M?" (id 0) (at 301.752 153.6699 0)
+    (property "Reference" "M2" (id 0) (at 302.26 153.6699 0)
       (effects (font (size 1.27 1.27)) (justify left))
     )
-    (property "Value" "Motor_DC" (id 1) (at 301.752 156.2099 0)
+    (property "Value" "Motor_DC" (id 1) (at 302.26 156.2099 0)
       (effects (font (size 1.27 1.27)) (justify left))
     )
@@
     )
     (path "/f8d8116b-49e3-4f76-99a7-2025425b0ac1"
-      (reference "M?") (unit 1) (value "Motor_DC") (footprint "")
+      (reference "M2") (unit 1) (value "Motor_DC") (footprint "")
     )
     (path "/2eb15ec9-1e13-430f-8e9b-31bd29a56841"
