File: Documentation/Electrical/Schematics/Sources/VisionSystem/VisionSystem.kicad_sch (KiCad schematic)
At the start: 13 parts

Commit message: update sch
Parts:
- gave numbers to parts that had none: 2
Changed lines of the file:
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@@
+    (stroke (width 0) (type default) (color 0 0 0 0))
+  )
+  (wire (pts (xy 341.63 157.988) (xy 341.63 159.512))
     (stroke (width 0) (type default) (color 0 0 0 0))
   )
@@
     (stroke (width 0) (type default) (color 0 0 0 0))
   )
+  (wire (pts (xy 341.63 168.656) (xy 341.63 166.116))
+    (stroke (width 0) (type default) (color 0 0 0 0))
+  )
   (wire (pts (xy 173.736 181.356) (xy 177.546 181.356))
     (stroke (width 0) (type default) (color 0 0 0 0))
@@
     (stroke (width 0) (type default) (color 0 0 0 0))
   )
+  (wire (pts (xy 326.644 159.512) (xy 341.63 159.512))
+    (stroke (width 0) (type default) (color 0 0 0 0))
+  )
   (wire (pts (xy 129.794 344.932) (xy 134.366 344.932))
     (stroke (width 0) (type default) (color 0 0 0 0))
@@
   )
   (wire (pts (xy 169.926 116.586) (xy 169.926 125.73))
+    (stroke (width 0) (type default) (color 0 0 0 0))
+  )
+  (wire (pts (xy 326.644 166.116) (xy 341.63 166.116))
     (stroke (width 0) (type default) (color 0 0 0 0))
   )
@@
     (effects (font (size 3 3)) (justify left bottom))
   )
+  (symbol (lib_id "power:GND") (at 341.63 168.656 0) (unit 1)
+    (in_bom yes) (on_board yes) (fields_autoplaced)
+    (property "Reference" "#PWR?" (id 0) (at 341.63 175.006 0)
+      (effects (font (size 1.27 1.27)) hide)
+    )
+    (property "Value" "GND" (id 1) (at 341.63 174.244 0))
+    (property "Footprint" "" (id 2) (at 341.63 168.656 0)
+      (effects (font (size 1.27 1.27)) hide)
+    )
+    (property "Datasheet" "" (id 3) (at 341.63 168.656 0)
+      (effects (font (size 1.27 1.27)) hide)
+    )
+    (pin "1")
+  )
   (symbol (lib_id "VL53L0X:VL53L0X") (at 152.146 135.89 0) (unit 1)
     (in_bom yes) (on_board yes) (fields_autoplaced)
-    (property "Reference" "U?" (id 0) (at 152.146 118.364 0))
-    (property "Value" "VL53L0X" (id 1) (at 152.146 120.904 0))
+    (property "Reference" "ToFLIDAR" (id 0) (at 152.146 118.11 0))
+    (property "Value" "VL53L0X" (id 1) (at 152.146 120.65 0))
     (property "Footprint" "SENSOR_VL53L0X" (id 2) (at 152.146 135.89 0)
       (effects (font (size 1.27 1.27)) (justify bottom) hide)
@@
   (symbol (lib_id "VL53L0X:VL53L0X") (at 152.146 276.86 0) (unit 1)
     (in_bom yes) (on_board yes) (fields_autoplaced)
-    (property "Reference" "U?" (id 0) (at 152.146 259.334 0))
-    (property "Value" "VL53L0X" (id 1) (at 152.146 261.874 0))
+    (property "Reference" "ToFLIDAR" (id 0) (at 152.146 259.08 0))
+    (property "Value" "VL53L0X" (id 1) (at 152.146 261.62 0))
     (property "Footprint" "SENSOR_VL53L0X" (id 2) (at 152.146 276.86 0)
       (effects (font (size 1.27 1.27)) (justify bottom) hide)
@@
     (pin "9")
   )
+  (symbol (lib_id "power:+5V") (at 341.63 157.988 0) (unit 1)
+    (in_bom yes) (on_board yes) (fields_autoplaced)
+    (property "Reference" "#PWR?" (id 0) (at 341.63 161.798 0)
+      (effects (font (size 1.27 1.27)) hide)
+    )
+    (property "Value" "+5V" (id 1) (at 341.63 152.4 0))
+    (property "Footprint" "" (id 2) (at 341.63 157.988 0)
+      (effects (font (size 1.27 1.27)) hide)
+    )
+    (property "Datasheet" "" (id 3) (at 341.63 157.988 0)
+      (effects (font (size 1.27 1.27)) hide)
+    )
+    (pin "1")
+  )
   (symbol (lib_id "TCS34725FN:TCS34725FN") (at 230.632 99.06 0) (unit 1)
-    (in_bom yes) (on_board yes) (fields_autoplaced)
-    (property "Reference" "U?" (id 0) (at 230.632 83.82 0))
+    (in_bom yes) (on_board yes)
+    (property "Reference" "ColorSensor" (id 0) (at 230.632 83.82 0))
     (property "Value" "TCS34725FN" (id 1) (at 230.632 86.36 0))
     (property "Footprint" "SON65P200X240X70-6N" (id 2) (at 230.632 99.06 0)
@@
   (symbol (lib_id "VL53L0X:VL53L0X") (at 152.146 102.108 0) (unit 1)
     (in_bom yes) (on_board yes) (fields_autoplaced)
-    (property "Reference" "U?" (id 0) (at 152.146 84.582 0))
-    (property "Value" "VL53L0X" (id 1) (at 152.146 87.122 0))
+    (property "Reference" "ToFLIDAR" (id 0) (at 152.146 83.82 0))
+    (property "Value" "VL53L0X" (id 1) (at 152.146 86.36 0))
     (property "Footprint" "SENSOR_VL53L0X" (id 2) (at 152.146 102.108 0)
       (effects (font (size 1.27 1.27)) (justify bottom) hide)
@@
   (symbol (lib_id "VL53L0X:VL53L0X") (at 152.146 206.502 0) (unit 1)
     (in_bom yes) (on_board yes) (fields_autoplaced)
-    (property "Reference" "U?" (id 0) (at 152.146 188.976 0))
-    (property "Value" "VL53L0X" (id 1) (at 152.146 191.516 0))
+    (property "Reference" "ToFLIDAR" (id 0) (at 152.146 189.23 0))
+    (property "Value" "VL53L0X" (id 1) (at 152.146 191.77 0))
     (property "Footprint" "SENSOR_VL53L0X" (id 2) (at 152.146 206.502 0)
       (effects (font (size 1.27 1.27)) (justify bottom) hide)
@@
   (symbol (lib_id "VL53L0X:VL53L0X") (at 152.146 171.196 0) (unit 1)
     (in_bom yes) (on_board yes) (fields_autoplaced)
-    (property "Reference" "U?" (id 0) (at 152.146 153.67 0))
+    (property "Reference" "ToFLIDAR" (id 0) (at 152.146 153.67 0))
     (property "Value" "VL53L0X" (id 1) (at 152.146 156.21 0))
     (property "Footprint" "SENSOR_VL53L0X" (id 2) (at 152.146 171.196 0)
@@
   (symbol (lib_id "VL53L0X:VL53L0X") (at 152.146 344.932 0) (unit 1)
     (in_bom yes) (on_board yes) (fields_autoplaced)
-    (property "Reference" "U?" (id 0) (at 152.146 327.406 0))
-    (property "Value" "VL53L0X" (id 1) (at 152.146 329.946 0))
+    (property "Reference" "ToFLIDAR" (id 0) (at 152.146 327.66 0))
+    (property "Value" "VL53L0X" (id 1) (at 152.146 330.2 0))
     (property "Footprint" "SENSOR_VL53L0X" (id 2) (at 152.146 344.932 0)
       (effects (font (size 1.27 1.27)) (justify bottom) hide)
@@
   (symbol (lib_id "VL53L0X:VL53L0X") (at 152.146 310.134 0) (unit 1)
     (in_bom yes) (on_board yes) (fields_autoplaced)
-    (property "Reference" "U?" (id 0) (at 152.146 292.608 0))
-    (property "Value" "VL53L0X" (id 1) (at 152.146 295.148 0))
+    (property "Reference" "ToFLIDAR" (id 0) (at 152.146 292.1 0))
+    (property "Value" "VL53L0X" (id 1) (at 152.146 294.64 0))
     (property "Footprint" "SENSOR_VL53L0X" (id 2) (at 152.146 310.134 0)
       (effects (font (size 1.27 1.27)) (justify bottom) hide)
@@
   (symbol (lib_id "TCS34725FN:TCS34725FN") (at 230.886 128.27 0) (unit 1)
     (in_bom yes) (on_board yes) (fields_autoplaced)
-    (property "Reference" "U?" (id 0) (at 230.886 113.03 0))
+    (property "Reference" "ColorSensor" (id 0) (at 230.886 113.03 0))
     (property "Value" "TCS34725FN" (id 1) (at 230.886 115.57 0))
     (property "Footprint" "SON65P200X240X70-6N" (id 2) (at 230.886 128.27 0)
@@
   (symbol (lib_id "VL53L0X:VL53L0X") (at 152.146 241.554 0) (unit 1)
     (in_bom yes) (on_board yes) (fields_autoplaced)
-    (property "Reference" "U?" (id 0) (at 152.146 224.028 0))
-    (property "Value" "VL53L0X" (id 1) (at 152.146 226.568 0))
+    (property "Reference" "ToFLIDAR" (id 0) (at 152.146 223.52 0))
+    (property "Value" "VL53L0X" (id 1) (at 152.146 226.06 0))
     (property "Footprint" "SENSOR_VL53L0X" (id 2) (at 152.146 241.554 0)
       (effects (font (size 1.27 1.27)) (justify bottom) hide)
@@
   )
   (symbol_instances
+    (path "/0820a483-5e6f-4694-9ab0-e79e7f9775f5"
+      (reference "#PWR?") (unit 1) (value "GND") (footprint "")
+    )
     (path "/2e1e6281-0991-4814-9e62-4e28c44fa195"
       (reference "#PWR?") (unit 1) (value "GND") (footprint "")
     )
+    (path "/326a4693-fdaa-4642-9895-c43c0f658e2d"
+      (reference "#PWR?") (unit 1) (value "+5V") (footprint "")
+    )
+    (path "/32d751f8-11e3-4e5f-94a9-837d86bd5921"
+      (reference "ColorSensor") (unit 1) (value "TCS34725FN") (footprint "SON65P200X240X70-6N")
+    )
+    (path "/e97be832-68f2-43bf-81a7-6e394c03766a"
+      (reference "ColorSensor") (unit 1) (value "TCS34725FN") (footprint "SON65P200X240X70-6N")
+    )
     (path "/c7802c66-6b6a-461f-bc05-285167d43bca"
       (reference "J?") (unit 1) (value "Jetson Nano 40 pin Header") (footprint "")
@@
     )
     (path "/12c943ec-a0d1-4282-a073-8e9c93908e26"
-      (reference "U?") (unit 1) (value "VL53L0X") (footprint "SENSOR_VL53L0X")
+      (reference "ToFLIDAR") (unit 1) (value "VL53L0X") (footprint "SENSOR_VL53L0X")
     )
     (path "/2f85c952-6da9-44a9-9339-38980ffdf8de"
-      (reference "U?") (unit 1) (value "VL53L0X") (footprint "SENSOR_VL53L0X")
-    )
-    (path "/32d751f8-11e3-4e5f-94a9-837d86bd5921"
-      (reference "U?") (unit 1) (value "TCS34725FN") (footprint "SON65P200X240X70-6N")
+      (reference "ToFLIDAR") (unit 1) (value "VL53L0X") (footprint "SENSOR_VL53L0X")
     )
     (path "/6617613f-da39-4d0e-8092-9a140925c9d4"
-      (reference "U?") (unit 1) (value "VL53L0X") (footprint "SENSOR_VL53L0X")
+      (reference "ToFLIDAR") (unit 1) (value "VL53L0X") (footprint "SENSOR_VL53L0X")
     )
     (path "/982c4c47-8236-4ef0-84ad-0709ed262982"
-      (reference "U?") (unit 1) (value "VL53L0X") (footprint "SENSOR_VL53L0X")
+      (reference "ToFLIDAR") (unit 1) (value "VL53L0X") (footprint "SENSOR_VL53L0X")
     )
     (path "/c1a4a996-3d02-40f9-b6f8-81d9b19b6076"
-      (reference "U?") (unit 1) (value "VL53L0X") (footprint "SENSOR_VL53L0X")
+      (reference "ToFLIDAR") (unit 1) (value "VL53L0X") (footprint "SENSOR_VL53L0X")
     )
     (path "/ce833cfd-ea31-45a2-a928-df93d4d84c7a"
-      (reference "U?") (unit 1) (value "VL53L0X") (footprint "SENSOR_VL53L0X")
+      (reference "ToFLIDAR") (unit 1) (value "VL53L0X") (footprint "SENSOR_VL53L0X")
     )
     (path "/d4684460-1e53-4ee8-9c89-4e9c8077ceca"
-      (reference "U?") (unit 1) (value "VL53L0X") (footprint "SENSOR_VL53L0X")
-    )
-    (path "/e97be832-68f2-43bf-81a7-6e394c03766a"
-      (reference "U?") (unit 1) (value "TCS34725FN") (footprint "SON65P200X240X70-6N")
+      (reference "ToFLIDAR") (unit 1) (value "VL53L0X") (footprint "SENSOR_VL53L0X")
     )
     (path "/f1cd1fa4-8d83-4c1c-818e-47dc0e358a24"
-      (reference "U?") (unit 1) (value "VL53L0X") (footprint "SENSOR_VL53L0X")
-    )
-  )
+      (reference "ToFLIDAR") (unit 1) (value "VL53L0X") (footprint "SENSOR_VL53L0X")
+    )
+  )
